File: pcb/ESPFanController.kicad_sch (KiCad schematic)
At the start: 19 parts, among them J1 Serial, J2 12Vin, M1 Fan1, M2 Fan2, M3 Fan3, SW1 Boot, U1 AMS1117-3.3, U2 ESP32-WROOM-32

Commit message: feat: add position for pullups
Parts:
- added R7, R8: 4k7, Resistor_SMD:R_0402_1005Metric_Pad0.72x0.64mm_HandSolder, symbol Device:R_Small
Connections:
- net +3V3: now also R7.1, R8.1
- net RX: now also R7.2
- net TX: now also R8.2

Commit message: feat: add second LED
feat: add cutouts to the corners

feat: add optional pull-ups to serial pins
  for I2C use after programming
Parts:
- added D2: Yellow, LED_SMD:LED_0603_1608Metric, symbol Device:LED_Small
- added R9: 680R, Resistor_SMD:R_0402_1005Metric, symbol Device:R_Small
- C1: LCSC (none) -> C15525
- C2: LCSC (none) -> C1525
- C3, C4: LCSC (none) -> C7171
- D1: value LED_Small -> Red; LCSC (none) -> C2286
- J1: LCSC (none) -> C131334
- R1, R2, R3, R4, R5: LCSC (none) -> C25744
- R6: LCSC (none) -> C25130
- R7, R8: LCSC (none) -> C25900
- SW1: LCSC (none) -> C318884
- U1: LCSC (none) -> C6186
- U2: LCSC (none) -> C701341
Connections:
- net GND: now also R9.2
- net Yellow: now reaches U2.36 (IO22)
- net Yellow: now also D2.2 (A)
- net LED renamed Red
- new net: D2.1 (K), R9.1
- no-connect marks 23 -> 22
